Commit message: joinz ug fix

File: mecanumbot_description/urdf/mecanumbot.urdf (robot description, URDF)
Before this commit: robot mecanumbot, 14 links, 13 joints
Joints:
- joint ${namespace}grabber_left_joint: limit lower=-1.57 upper=1.57 -> lower=-1.57 upper=1.57 effort=5.0 velocity=1.0
- joint ${namespace}grabber_right_joint: limit lower=-1.57 upper=1.57 -> lower=-1.57 upper=1.57 effort=5.0 velocity=1.0
- joint ${namespace}head_joint: limit lower=-1.57 upper=0.52 -> lower=-1.57 upper=1.57 effort=5.0 velocity=1.0

Commit message: no namespace in description

File: mecanumbot_description/urdf/mecanumbot.urdf (robot description, URDF)
Before this commit: robot mecanumbot, 14 links, 13 joints
Links:
- removed link ${namespace}base_footprint
- removed link ${namespace}base_link
- removed link ${namespace}base_scan
- removed link ${namespace}camera_link
- removed link ${namespace}camera_rgb_frame
- removed link ${namespace}camera_rgb_optical_frame
- removed link ${namespace}grabber_left_link
- removed link ${namespace}grabber_right_link
- removed link ${namespace}head_link
- removed link ${namespace}imu_link
- removed link ${namespace}wheel_backleft_link
- removed link ${namespace}wheel_backright_link
- removed link ${namespace}wheel_frontleft_link
- removed link ${namespace}wheel_frontright_link
- added link base_footprint
- added link base_link; collision box size=0.045 0.260 0.09; collision box size=0.2 0.2 0.2
- added link base_scan, mass 0.114; collision cylinder length=0.0315 radius=0.055; visual mesh filename=package://mecanumbot_description/meshes/lds.stl scale=0.001 0.001 0.001
- added link camera_link; collision box size=0.015 0.030 0.027; visual box size=0.015 0.030 0.027
- added link camera_rgb_frame
- added link camera_rgb_optical_frame
- added link grabber_left_link; collision mesh filename=package://mecanumbot_description/meshes/arm_left.stl scale=0.001 0.001 0.001; visual mesh filename=package://mecanumbot_description/meshes/arm_left.stl scale=0.001 0.001 0.001
- added link grabber_right_link; collision mesh filename=package://mecanumbot_description/meshes/arm_right.stl scale=0.001 0.001 0.001; visual mesh filename=package://mecanumbot_description/meshes/arm_right.stl scale=0.001 0.001 0.001
- added link head_link; visual mesh filename=package://mecanumbot_description/meshes/head.stl scale=0.001 0.001 0.001
- added link imu_link
- added link wheel_backleft_link; collision cylinder length=0.030 radius=0.033; visual mesh filename=package://mecanumbot_description/meshes/wheel.stl scale=0.001 0.001 0.001
- added link wheel_backright_link; collision cylinder length=0.030 radius=0.033; visual mesh filename=package://mecanumbot_description/meshes/wheel.stl scale=0.001 0.001 0.001
- added link wheel_frontleft_link; collision cylinder length=0.030 radius=0.033; visual mesh filename=package://mecanumbot_description/meshes/wheel.stl scale=0.001 0.001 0.001
- added link wheel_frontright_link; collision cylinder length=0.030 radius=0.033; visual mesh filename=package://mecanumbot_description/meshes/wheel.stl scale=0.001 0.001 0.001
Joints:
- removed joint ${namespace}base_joint
- removed joint ${namespace}camera_joint
- removed joint ${namespace}camera_rgb_joint
- removed joint ${namespace}camera_rgb_optical_joint
- removed joint ${namespace}grabber_left_joint
- removed joint ${namespace}grabber_right_joint
- removed joint ${namespace}head_joint
- removed joint ${namespace}imu_joint
- removed joint ${namespace}scan_joint
- removed joint ${namespace}wheel_backleft_joint
- removed joint ${namespace}wheel_backright_joint
- removed joint ${namespace}wheel_frontleft_joint
- removed joint ${namespace}wheel_frontright_joint
- added joint base_joint: type fixed, parent base_footprint, child base_link, origin xyz=0.0 0.0 0.01 rpy=0 0 0
- added joint camera_joint: type fixed, parent head_link, child camera_link, origin xyz=0.022 0.038 0.0 rpy=0 0 0
- added joint camera_rgb_joint: type fixed, parent camera_link, child camera_rgb_frame, origin xyz=0.003 0.011 0.009 rpy=0 0 0
- added joint camera_rgb_optical_joint: type fixed, parent camera_rgb_frame, child camera_rgb_optical_frame, origin xyz=0 0 0 rpy=-1.57 0 -1.57
- added joint grabber_left_joint: type revolute, parent base_link, child grabber_left_link, origin xyz=0.174 0.070 0.024 rpy=0 0 0, axis 0 0 1, limit lower=-1.57 upper=1.57 effort=5.0 velocity=1.0
- added joint grabber_right_joint: type revolute, parent base_link, child grabber_right_link, origin xyz=0.174 -0.070 0.024 rpy=0 0 0, axis 0 0 1, limit lower=-1.57 upper=1.57 effort=5.0 velocity=1.0
- added joint head_joint: type revolute, parent base_link, child head_link, origin xyz=0.1063 0.0 0.1679 rpy=1.57 0 0, axis 0 0 1, limit lower=-1.57 upper=1.57 effort=5.0 velocity=1.0
- added joint imu_joint: type fixed, parent base_link, child imu_link, origin xyz=0.0 0 0.068 rpy=0 0 0
- added joint scan_joint: type fixed, parent base_link, child base_scan, origin xyz=0 0 0.122 rpy=0 0 0
- added joint wheel_backleft_joint: type continuous, parent base_link, child wheel_backleft_link, origin xyz=-0.064 0.1522 0.02345 rpy=-1.57 0 0, axis 0 0 1
- added joint wheel_backright_joint: type continuous, parent base_link, child wheel_backright_link, origin xyz=-0.064 -0.1522 0.02345 rpy=1.57 0 0, axis 0 0 1
- added joint wheel_frontleft_joint: type continuous, parent base_link, child wheel_frontleft_link, origin xyz=0.064 0.1522 0.02345 rpy=-1.57 0 0, axis 0 0 1
- added joint wheel_frontright_joint: type continuous, parent base_link, child wheel_frontright_link, origin xyz=0.064 -0.1522 0.02345 rpy=1.57 0 0, axis 0 0 1

Commit message: urdf with relative path

File: mecanumbot_description/urdf/mecanumbot.urdf (robot description, URDF)
Before this commit: robot mecanumbot, 14 links, 13 joints
Links:
- link base_link: geometry collision box size=0.045 0.260 0.09; collision box size=0.2 0.2 0.2
- link base_scan: geometry collision cylinder length=0.0315 radius=0.055; visual mesh filename=../meshes/lds.stl scale=0.001 0.001 0.001
- link grabber_left_link: geometry collision mesh filename=../meshes/arm_left.STL scale=0.001 0.001 0.001; visual mesh filename=../meshes/arm_left.STL scale=0.001 0.001 0.001
- link grabber_right_link: geometry collision mesh filename=../meshes/arm_right.STL scale=0.001 0.001 0.001; visual mesh filename=../meshes/arm_right.STL scale=0.001 0.001 0.001
- link head_link: geometry visual mesh filename=../meshes/head.STL scale=0.001 0.001 0.001
- link wheel_backleft_link: geometry collision cylinder length=0.030 radius=0.033; visual mesh filename=../meshes/wheel.STL scale=0.001 0.001 0.001
- link wheel_backright_link: geometry collision cylinder length=0.030 radius=0.033; visual mesh filename=../meshes/wheel.STL scale=0.001 0.001 0.001
- link wheel_frontleft_link: geometry collision cylinder length=0.030 radius=0.033; visual mesh filename=../meshes/wheel.STL scale=0.001 0.001 0.001
- link wheel_frontright_link: geometry collision cylinder length=0.030 radius=0.033; visual mesh filename=../meshes/wheel.STL scale=0.001 0.001 0.001

Commit message: urdf namespace added and path

File: mecanumbot_description/urdf/mecanumbot.urdf (robot description, URDF)
Before this commit: robot mecanumbot, 14 links, 13 joints
Links:
- removed link base_footprint
- removed link base_link
- removed link base_scan
- removed link camera_link
- removed link camera_rgb_frame
- removed link camera_rgb_optical_frame
- removed link grabber_left_link
- removed link grabber_right_link
- removed link head_link
- removed link imu_link
- removed link wheel_backleft_link
- removed link wheel_backright_link
- removed link wheel_frontleft_link
- removed link wheel_frontright_link
- added link ${namespace}base_footprint
- added link ${namespace}base_link; collision box size=0.045 0.260 0.09; collision box size=0.2 0.2 0.2
- added link ${namespace}base_scan, mass 0.114; collision cylinder length=0.0315 radius=0.055; visual mesh filename=package://mecanumbot_description/meshes/lds.stl scale=0.001 0.001 0.001
- added link ${namespace}camera_link; collision box size=0.015 0.030 0.027; visual box size=0.015 0.030 0.027
- added link ${namespace}camera_rgb_frame
- added link ${namespace}camera_rgb_optical_frame
- added link ${namespace}grabber_left_link; collision mesh filename=package://mecanumbot_description/meshes/arm_left.STL scale=0.001 0.001 0.001; visual mesh filename=package://mecanumbot_description/meshes/arm_left.STL scale=0.001 0.001 0.001
- added link ${namespace}grabber_right_link; collision mesh filename=package://mecanumbot_description/meshes/arm_right.STL scale=0.001 0.001 0.001; visual mesh filename=package://mecanumbot_description/meshes/arm_right.STL scale=0.001 0.001 0.${namespace}001
- added link ${namespace}head_link; visual mesh filename=package://mecanumbot_description/meshes/head.STL scale=0.001 0.001 0.001
- added link ${namespace}imu_link
- added link ${namespace}wheel_backleft_link; collision cylinder length=0.030 radius=0.033; visual mesh filename=package://mecanumbot_description/meshes/wheel.STL scale=0.001 0.001 0.001
- added link ${namespace}wheel_backright_link; collision cylinder length=0.030 radius=0.033; visual mesh filename=package://mecanumbot_description/meshes/wheel.STL scale=0.001 0.001 0.001
- added link ${namespace}wheel_frontleft_link; collision cylinder length=0.030 radius=0.033; visual mesh filename=package://mecanumbot_description/meshes/wheel.STL scale=0.001 0.001 0.001
- added link ${namespace}wheel_frontright_link; collision cylinder length=0.030 radius=0.033; visual mesh filename=package://mecanumbot_description/meshes/wheel.STL scale=0.001 0.001 0.001
Joints:
- removed joint base_joint
- removed joint camera_joint
- removed joint camera_rgb_joint
- removed joint camera_rgb_optical_joint
- removed joint grabber_left_joint
- removed joint grabber_right_joint
- removed joint head_joint
- removed joint imu_joint
- removed joint scan_joint
- removed joint wheel_backleft_joint
- removed joint wheel_backright_joint
- removed joint wheel_frontleft_joint
- removed joint wheel_frontright_joint
- added joint ${namespace}base_joint: type fixed, parent ${namespace}base_footprint, child ${namespace}base_link, origin xyz=0.0 0.0 0.01 rpy=0 0 0
- added joint ${namespace}camera_joint: type fixed, parent ${namespace}head_link, child ${namespace}camera_link, origin xyz=0.022 0.038 0.0 rpy=0 0 0
- added joint ${namespace}camera_rgb_joint: type fixed, parent ${namespace}camera_link, child ${namespace}camera_rgb_frame, origin xyz=0.003 0.011 0.009 rpy=0 0 0
- added joint ${namespace}camera_rgb_optical_joint: type fixed, parent ${namespace}camera_rgb_frame, child ${namespace}camera_rgb_optical_frame, origin xyz=0 0 0 rpy=-1.57 0 -1.57
- added joint ${namespace}grabber_left_joint: type revolute, parent ${namespace}base_link, child ${namespace}grabber_left_link, origin xyz=0.174 0.070 0.024 rpy=0 0 0, axis 0 0 1, limit lower=-1.57 upper=1.57 effort=5.0 velocity=1.0
- added joint ${namespace}grabber_right_joint: type revolute, parent ${namespace}base_link, child ${namespace}grabber_right_link, origin xyz=0.174 -0.070 0.024 rpy=0 0 0, axis 0 0 1, limit lower=-1.57 upper=1.57 effort=5.0 velocity=1.0
- added joint ${namespace}head_joint: type revolute, parent ${namespace}base_link, child ${namespace}head_link, origin xyz=0.1063 0.0 0.1679 rpy=1.57 0 0, axis 0 0 1, limit lower=-1.57 upper=1.57 effort=5.0 velocity=1.0
- added joint ${namespace}imu_joint: type fixed, parent ${namespace}base_link, child ${namespace}imu_link, origin xyz=0.0 0 0.068 rpy=0 0 0
- added joint ${namespace}scan_joint: type fixed, parent ${namespace}base_link, child ${namespace}base_scan, origin xyz=0 0 0.122 rpy=0 0 0
- added joint ${namespace}wheel_backleft_joint: type continuous, parent ${namespace}base_link, child ${namespace}wheel_backleft_link, origin xyz=-0.064 0.1522 0.02345 rpy=-1.57 0 0, axis 0 0 1
- added joint ${namespace}wheel_backright_joint: type continuous, parent base_link, child wheel_backright_link, origin xyz=-0.064 -0.1522 0.02345 rpy=1.57 0 0, axis 0 0 1
- added joint ${namespace}wheel_frontleft_joint: type continuous, parent ${namespace}base_link, child ${namespace}wheel_frontleft_link, origin xyz=0.064 0.1522 0.02345 rpy=-1.57 0 0, axis 0 0 1
- added joint ${namespace}wheel_frontright_joint: type continuous, parent ${namespace}base_link, child ${namespace}wheel_frontright_link, origin xyz=0.064 -0.1522 0.02345 rpy=1.57 0 0, axis 0 0 1

Commit message: parameters set, urdf fixed

File: mecanumbot_description/urdf/mecanumbot.urdf (robot description, URDF)
Before this commit: robot mecanumbot, 14 links, 13 joints
Links:
- link ${namespace}base_link: geometry collision box size=0.045 0.260 0.09; collision box size=0.2 0.2 0.2
- link ${namespace}grabber_left_link: geometry collision mesh filename=package://mecanumbot_description/meshes/arm_left.stl scale=0.001 0.001 0.001; visual mesh filename=package://mecanumbot_description/meshes/arm_left.stl scale=0.001 0.001 0.001
- link ${namespace}grabber_right_link: geometry collision mesh filename=package://mecanumbot_description/meshes/arm_right.stl scale=0.001 0.001 0.001; visual mesh filename=package://mecanumbot_description/meshes/arm_right.stl scale=0.001 0.001 0.${namespace}001
- link ${namespace}head_link: geometry visual mesh filename=package://mecanumbot_description/meshes/head.stl scale=0.001 0.001 0.001
- link ${namespace}wheel_backleft_link: geometry collision cylinder length=0.030 radius=0.033; visual mesh filename=package://mecanumbot_description/meshes/wheel.stl scale=0.001 0.001 0.001
- link ${namespace}wheel_backright_link: geometry collision cylinder length=0.030 radius=0.033; visual mesh filename=package://mecanumbot_description/meshes/wheel.stl scale=0.001 0.001 0.001
- link ${namespace}wheel_frontleft_link: geometry collision cylinder length=0.030 radius=0.033; visual mesh filename=package://mecanumbot_description/meshes/wheel.stl scale=0.001 0.001 0.001
- link ${namespace}wheel_frontright_link: geometry collision cylinder length=0.030 radius=0.033; visual mesh filename=package://mecanumbot_description/meshes/wheel.stl scale=0.001 0.001 0.001

Commit message: Fix namespace issues
Remove wrong namespace declaration and add missing ones in URDF
Fix namespace declaration in state_publisher's launch

File: mecanumbot_description/urdf/mecanumbot.urdf (robot description, URDF)
Before this commit: robot mecanumbot, 14 links, 13 joints
Links:
- link ${namespace}grabber_right_link: geometry collision mesh filename=package://mecanumbot_description/meshes/arm_right.stl scale=0.001 0.001 0.001; visual mesh filename=package://mecanumbot_description/meshes/arm_right.stl scale=0.001 0.001 0.001
Joints:
- joint ${namespace}wheel_backright_joint: child wheel_backright_link -> ${namespace}wheel_backright_link; parent base_link -> ${namespace}base_link

Commit message: Make link namespace pretty - Csenge
add / to namespaces so that it does not get melted into the names

File: mecanumbot_description/urdf/mecanumbot.urdf (robot description, URDF)
Before this commit: robot mecanumbot, 14 links, 13 joints
Links:
- removed link ${namespace}base_footprint
- removed link ${namespace}base_link
- removed link ${namespace}base_scan
- removed link ${namespace}camera_link
- removed link ${namespace}camera_rgb_frame
- removed link ${namespace}camera_rgb_optical_frame
- removed link ${namespace}grabber_left_link
- removed link ${namespace}grabber_right_link
- removed link ${namespace}head_link
- removed link ${namespace}imu_link
- removed link ${namespace}wheel_backleft_link
- removed link ${namespace}wheel_backright_link
- removed link ${namespace}wheel_frontleft_link
- removed link ${namespace}wheel_frontright_link
- added link ${namespace}/base_footprint
- added link ${namespace}/base_link; collision box size=0.045 0.260 0.09; collision box size=0.2 0.2 0.2
- added link ${namespace}/base_scan, mass 0.114; collision cylinder length=0.0315 radius=0.055; visual mesh filename=package://mecanumbot_description/meshes/lds.stl scale=0.001 0.001 0.001
- added link ${namespace}/camera_link; collision box size=0.015 0.030 0.027; visual box size=0.015 0.030 0.027
- added link ${namespace}/camera_rgb_frame
- added link ${namespace}/camera_rgb_optical_frame
- added link ${namespace}/grabber_left_link; collision mesh filename=package://mecanumbot_description/meshes/arm_left.stl scale=0.001 0.001 0.001; visual mesh filename=package://mecanumbot_description/meshes/arm_left.stl scale=0.001 0.001 0.001
- added link ${namespace}/grabber_right_link; collision mesh filename=package://mecanumbot_description/meshes/arm_right.stl scale=0.001 0.001 0.001; visual mesh filename=package://mecanumbot_description/meshes/arm_right.stl scale=0.001 0.001 0.001
- added link ${namespace}/head_link; visual mesh filename=package://mecanumbot_description/meshes/head.stl scale=0.001 0.001 0.001
- added link ${namespace}/imu_link
- added link ${namespace}/wheel_backleft_link; collision cylinder length=0.030 radius=0.033; visual mesh filename=package://mecanumbot_description/meshes/wheel.stl scale=0.001 0.001 0.001
- added link ${namespace}/wheel_backright_link; collision cylinder length=0.030 radius=0.033; visual mesh filename=package://mecanumbot_description/meshes/wheel.stl scale=0.001 0.001 0.001
- added link ${namespace}/wheel_frontleft_link; collision cylinder length=0.030 radius=0.033; visual mesh filename=package://mecanumbot_description/meshes/wheel.stl scale=0.001 0.001 0.001
- added link ${namespace}/wheel_frontright_link; collision cylinder length=0.030 radius=0.033; visual mesh filename=package://mecanumbot_description/meshes/wheel.stl scale=0.001 0.001 0.001
Joints:
- removed joint ${namespace}base_joint
- removed joint ${namespace}camera_joint
- removed joint ${namespace}camera_rgb_joint
- removed joint ${namespace}camera_rgb_optical_joint
- removed joint ${namespace}grabber_left_joint
- removed joint ${namespace}grabber_right_joint
- removed joint ${namespace}head_joint
- removed joint ${namespace}imu_joint
- removed joint ${namespace}scan_joint
- removed joint ${namespace}wheel_backleft_joint
- removed joint ${namespace}wheel_backright_joint
- removed joint ${namespace}wheel_frontleft_joint
- removed joint ${namespace}wheel_frontright_joint
- added joint ${namespace}/base_joint: type fixed, parent ${namespace}/base_footprint, child ${namespace}/base_link, origin xyz=0.0 0.0 0.01 rpy=0 0 0
- added joint ${namespace}/camera_joint: type fixed, parent ${namespace}/head_link, child ${namespace}/camera_link, origin xyz=0.022 0.038 0.0 rpy=0 0 0
- added joint ${namespace}/camera_rgb_joint: type fixed, parent ${namespace}/camera_link, child ${namespace}/camera_rgb_frame, origin xyz=0.003 0.011 0.009 rpy=0 0 0
- added joint ${namespace}/camera_rgb_optical_joint: type fixed, parent ${namespace}/camera_rgb_frame, child ${namespace}/camera_rgb_optical_frame, origin xyz=0 0 0 rpy=-1.57 0 -1.57
- added joint ${namespace}/grabber_left_joint: type revolute, parent ${namespace}/base_link, child ${namespace}/grabber_left_link, origin xyz=0.174 0.070 0.024 rpy=0 0 0, axis 0 0 1, limit lower=-1.57 upper=1.57 effort=5.0 velocity=1.0
- added joint ${namespace}/grabber_right_joint: type revolute, parent ${namespace}/base_link, child ${namespace}/grabber_right_link, origin xyz=0.174 -0.070 0.024 rpy=0 0 0, axis 0 0 1, limit lower=-1.57 upper=1.57 effort=5.0 velocity=1.0
- added joint ${namespace}/head_joint: type revolute, parent ${namespace}/base_link, child ${namespace}/head_link, origin xyz=0.1063 0.0 0.1679 rpy=1.57 0 0, axis 0 0 1, limit lower=-1.57 upper=1.57 effort=5.0 velocity=1.0
- added joint ${namespace}/imu_joint: type fixed, parent ${namespace}/base_link, child ${namespace}/imu_link, origin xyz=0.0 0 0.068 rpy=0 0 0
- added joint ${namespace}/scan_joint: type fixed, parent ${namespace}/base_link, child ${namespace}/base_scan, origin xyz=0 0 0.122 rpy=0 0 0
- added joint ${namespace}/wheel_backleft_joint: type continuous, parent ${namespace}/base_link, child ${namespace}/wheel_backleft_link, origin xyz=-0.064 0.1522 0.02345 rpy=-1.57 0 0, axis 0 0 1
- added joint ${namespace}/wheel_backright_joint: type continuous, parent ${namespace}/base_link, child ${namespace}/wheel_backright_link, origin xyz=-0.064 -0.1522 0.02345 rpy=1.57 0 0, axis 0 0 1
- added joint ${namespace}/wheel_frontleft_joint: type continuous, parent ${namespace}/base_link, child ${namespace}/wheel_frontleft_link, origin xyz=0.064 0.1522 0.02345 rpy=-1.57 0 0, axis 0 0 1
- added joint ${namespace}/wheel_frontright_joint: type continuous, parent ${namespace}/base_link, child ${namespace}/wheel_frontright_link, origin xyz=0.064 -0.1522 0.02345 rpy=1.57 0 0, axis 0 0 1
