Commit message: introduce flp of motor to urdf

File: mecanumbot_description/urdf/mecanumbot.urdf (robot description, URDF)
Before this commit: robot mecanumbot, 14 links, 13 joints
Joints:
- joint ${namespace}/camera_joint: origin xyz=0.022 0.038 0.0 rpy=0 0 0 -> xyz=0.022 0.038 0.0 rpy=0 -1.57 0

Commit message: fix frames

File: mecanumbot_description/urdf/mecanumbot.urdf (robot description, URDF)
Before this commit: robot mecanumbot, 14 links, 13 joints
Links:
- link ${namespace}/camera_link: geometry collision box size=0.027 0.015 0.030; visual box size=0.027 0.015 0.030
Joints:
- joint ${namespace}/camera_joint: origin xyz=0.022 0.038 0.0 rpy=0 -1.57 0 -> xyz=0.022 0.038 0.0 rpy=-1.5708 0 0
- joint ${namespace}/camera_rgb_joint: origin xyz=0.003 0.011 0.009 rpy=0 0 0 -> xyz=-0.009 -0.003 0.011 rpy=0 0 0

Commit message: update urdf

File: mecanumbot_description/urdf/mecanumbot.urdf (robot description, URDF)
Before this commit: robot mecanumbot, 14 links, 13 joints
Joints:
- joint ${namespace}/camera_joint: origin xyz=0.022 0.038 0.0 rpy=-1.5708 0 0 -> xyz=0.022 0.0545 0.0 rpy=-1.5708 0 0
- joint ${namespace}/camera_rgb_joint: origin xyz=-0.009 -0.003 0.011 rpy=0 0 0 -> xyz=0.0 0.0 0.0 rpy=0 0 0
- joint ${namespace}/head_joint: origin xyz=0.1063 0.0 0.1679 rpy=1.57 0 0 -> xyz=0.1063 0.0 0.1700 rpy=1.57 0 0
